File: opamp_block/opamp_block.kicad_sch (KiCad schematic)
At the start: 12 parts

Commit message: Update opamp block KiCad files
Parts:
- added C_TIMER2: 10n, symbol Device:C
- added R_TIMER2: 91k, symbol Device:R
- added TP_TIMER2: (no value), symbol Connector:TestPoint
- C_REF2A: Fitted false -> true; now fitted
- U_REF: value ZERO_DRIFT_RRIO_TBD -> OPA333AID; footprint (none) -> Package_SO:SOIC-8_3.9x4.9mm_P1.27mm; symbol Simulation_SPICE:OPAMP -> EDU1_Block:OPA333AID; Manufacturer (none) -> Texas Instruments
Connections:
- net AUX_5V: now also U_REF.7 (V+); no longer U_REF.3 (V+)
- net agnd: now also C_TIMER2.2
- net vaa: now also R_TIMER2.1
- net REF_DIV: no longer names the net of C_REF1.1, R_REF1.2, R_REF2.1
- net REF_DIV: now also U_REF.3 (+); no longer U_REF.1 (+)
- net U_REF_OUT: no longer names the net of R_REFISO.1
- net U_REF_OUT: now also U_REF.6; no longer U_REF.5
- new net discharge2: C_TIMER2.1, R_TIMER2.2
- new net timer_out2: TP_TIMER2.1
Other:
- note added: "91k / 10n: nominal RC interval = 1.001 ms. 555 compatibility and autonomous oscillation unconfirmed. Ibrahim to confirm timer behavior and block ownership."
- note added: "INTEGRATION Import this sheet and its two children; wire all 10 border pins in the parent. Master owns chip, main supply entry/current break, scan header and ground tie. J_AUX supplies AUX_5V; connect its source return to board AGND. OPA333 SOIC-8: +IN 3, -IN 2, V+ 7, V- 4, OUT 6; pads 1/5/8 unused. REF feedback is sensed after R_REFISO; C_REF2A and C_REF2B are populated."
- note added: "OPAMP BLOCK / SHARED SUPPORT + 10-PIN EXTERNAL INTERFACE"
- note added: "REF buffer and supply decoupling"
- note added: "TIMER2 / assumed open-drain discharge"
- note removed: "8 hierarchical labels become border pins when this sheet is inserted into the master project."
- note removed: "INTEGRATION / BUILD NOTES - Master owns chip, bench VAA entry/current break, scan header and AGND/DGND tie. - AUX_5V enters at J_AUX; its bench return connects to the board AGND. - No global labels: child supplies and signals pass through sheet pins. - Keep all three schematic files together; footprints are intentionally empty. - Pin 48: OPAMP1 block label vs op2_inp signal name remains unresolve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"
- note removed: "OPAMP BLOCK / SHARED SUPPORT + EXTERNAL INTERFACE"
- title: Op-amp block | REF, AUX supply and 8-pin interface -> Op-amp block | Shared support and 10-pin interface
- moved on the sheet: C_AUX1, C_AUX2, C_REF1, C_REF2B, C_VAA1, C_VAA2, J_AUX, R_REF1, R_REF2, R_REFISO, U_REF
