File: opamp_block/opamp_ch1.kicad_sch (KiCad schematic)
At the start: 53 parts, among them J1_BSIG GENERATOR, J1_BV1 V1_BIAS, J1_DSIG GENERATOR, J1_V1C V1, J1_VC VC, U1_NULL ZERO_DRIFT_RRIO_TBD

Commit message: Update opamp block KiCad files
Parts:
- C1_CNULL: value TBD -> 22p; Fitted false -> true; now fitted
- C1_D1A, C1_D1B, R1_D1A, R1_D1B: value TBD-AD -> UNSPECIFIED; Open_Item (none) -> Fixture D value requires gain, impedance and test frequency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
- C1_D2, R1_D2: value TBD -> UNSPECIFIED; Open_Item (none) -> Fixture D value requires gain, impedance and test frequency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
- R1_C2: value TBD-AD -> 20M; Tolerance (none) -> 0.1%
- R1_CL: value TBD -> 2k
- U1_NULL: value ZERO_DRIFT_RRIO_TBD -> OPA333AID; footprint (none) -> Package_SO:SOIC-8_3.9x4.9mm_P1.27mm; symbol Simulation_SPICE:OPAMP -> EDU1_Block:OPA333AID; Manufacturer (none) -> Texas Instruments
Connections:
- net AUX_5V: now also U1_NULL.7 (V+); no longer U1_NULL.3 (V+)
- net CH1_A_INN: no longer names the net of JP1A_INN.1 (Pin_1), R1_A3A.2, SW1_A1.2 (B)
- net CH1_A_INP: no longer names the net of JP1A_INP.1 (Pin_1), R1_A3B.2, SW1_A2.2 (B)
- net CH1_A_NIP: no longer names the net of R1_A3B.1, R1_A4.2, SW1_A2.1 (A)
- net CH1_A_OUT: no longer names the net of JP1A_OUT.1 (Pin_1), R1_A2.2, TP1_EA0.1
- net CH1_A_SUM: no longer names the net of R1_A1.2, R1_A2.1, R1_A3A.1, SW1_A1.1 (A)
- net CH1_B_GJ: no longer names the net of JP1_BG.1 (Pin_1), R1_BG.2
- net CH1_B_INN: no longer names the net of JP1B_INN.1 (Pin_1), R1_BF.2, R1_BG.1
- net CH1_B_INP: no longer names the net of JP1B_INP.1 (Pin_1), R1_BBIAS.1, R1_BIN.2
- net CH1_B_OUT: no longer names the net of JP1B_OUT.1 (Pin_1), R1_BF.1, TP1_EB0.1
- net CH1_B_SIG: no longer names the net of C1_BAC.2, R1_BDIR.2, R1_BIN.1
- net CH1_B_SIGIN: no longer names the net of C1_BAC.1, J1_BSIG.1 (In), R1_BDIR.1
- net CH1_B_V1: no longer names the net of J1_BV1.1 (Pin_1), JP1_BG.2 (Pin_2), R1_BV1.2
- net CH1_C_INN: no longer names the net of JP1C_INN.1 (Pin_1), R1_C1A.2, R1_C2.1
- net CH1_C_INP: no longer names the net of JP1C_INP.1 (Pin_1), R1_C1B.2
- net CH1_C_LOOP: no longer names the net of JP1_C.2 (Pin_2), R1_C2.2
- net CH1_C_NULLOUT: no longer names the net of C1_CNULL.1, JP1_C.1 (Pin_1), TP1_EC0.1
- net CH1_C_NULLOUT: now also U1_NULL.6; no longer U1_NULL.5
- net CH1_C_OUT: no longer names the net of JP1C_OUT.1 (Pin_1), R1_CL.1, TP1_V2.1
- net CH1_C_OUT: now also U1_NULL.3 (+); no longer U1_NULL.1 (+)
- net CH1_C_VCN: no longer names the net of C1_CNULL.2, R1_CVC.2, U1_NULL.2 (-)
- net CH1_DSIG: no longer names the net of J1_DSIG.1 (In), R1_D2.2
- net CH1_D_INJ: no longer names the net of C1_D2.2, R1_D2.1
- net CH1_D_INN: no longer names the net of C1_D1A.1, JP1D_INN.1 (Pin_1), R1_D1A.2
- net CH1_D_INP: no longer names the net of C1_D1B.1, JP1D_INP.1 (Pin_1), R1_D1B.2
- net CH1_D_OUT: no longer names the net of C1_D2.1, JP1D_OUT.1 (Pin_1), R1_D1A.1, TP1_V0.1
- net CH1_V1TERM: no longer names the net of J1_V1C.1 (Pin_1), R1_CL.2
- net CH1_VCTERM: no longer names the net of J1_VC.1 (Pin_1), R1_CVC.1
- net CH1_VQI: no longer names the net of R1_A1.1, R1_A4.1, R1_AVQI.2, TP1_VQI.1
Other:
- note added: "A / Offset and input currents"
- note added: "B / Dynamic tests and quiescent current"
- note added: "BG open: follower; closed: gain about 101. AC option: remove BDIR, fit BAC and BBIAS."
- note added: "C / Null-loop gain and output swing"
- note added: "CNULL = 22 pF is a bring-up starting point. Servo feedback passes through the chip. Do not add a local feedback resistor around the null amplifier."
- note added: "Fixture D values remain open; all D parts stay unpopulated. Generator shields return to AGND. Offset applied stimuli relative to REF."
- note added: "Guard the high-impedance A nodes with REF. Switches remain independent."
- note added: "No board placement/routing. Fixture B PD/Iq is an engineering adaptation of Method 4005."
- note removed: "A / Vos, Ib, Ios"
- note removed: "All symbols retained with DNP flags. Values await AD / ZO / frequency. Coax shield returns to AGND; stimulus referenced/offset to REF."
- note removed: "B / Slew rate, phase margin, GBW, PD/Iq"
- note removed: "BUILD: silkscreen fixture letters beside isolation jumpers. TBD and TBD-AD are intentional. No PCB placement/routing. Fixture B PD/Iq is an EDU1 engineering adaptation, not literal Figure 4005-1 conformity."
- note removed: "C / Open-loop gain and output swing"
- note removed: "Guard CH1_A_SUM, CH1_A_INN, CH1_A_NIP, CH1_A_INP with REF. No vias inside guard; no solder-mask opening. Switches independent."
- note removed: "JP1_BG open: follower; closed: gain ~101. DC coupling default. AC option: remove R1_BDIR; fit C1_BAC and R1_BBIAS."
- note removed: "JP1_C closed for retained tests. Servo feedback passes through chip. R1_CVC fitted at 0 ohm; C1_CNULL DNP. Do not add local feedback."
- moved on the sheet: C1_BAC, C1_D1A, C1_D1B, C1_D2, J1_BSIG, J1_BV1, J1_DSIG, J1_V1C, J1_VC, JP1A_INN, JP1A_INP, JP1A_OUT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
