File: opamp_block/opamp_ch2.kicad_sch (KiCad schematic)
At the start: 53 parts, among them J2_BSIG GENERATOR, J2_BV1 V1_BIAS, J2_DSIG GENERATOR, J2_V1C V1, J2_VC VC, U2_NULL ZERO_DRIFT_RRIO_TBD

Commit message: Update opamp block KiCad files
Parts:
- C2_CNULL: value TBD -> 22p; Fitted false -> true; now fitted
- C2_D1A, C2_D1B, R2_D1A, R2_D1B: value TBD-AD -> UNSPECIFIED; Open_Item (none) -> Fixture D value requires gain, impedance and test frequency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
- C2_D2, R2_D2: value TBD -> UNSPECIFIED; Open_Item (none) -> Fixture D value requires gain, impedance and test frequency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
- R2_C2: value TBD-AD -> 20M; Tolerance (none) -> 0.1%
- R2_CL: value TBD -> 2k
- U2_NULL: value ZERO_DRIFT_RRIO_TBD -> OPA333AID; footprint (none) -> Package_SO:SOIC-8_3.9x4.9mm_P1.27mm; symbol Simulation_SPICE:OPAMP -> EDU1_Block:OPA333AID; Manufacturer (none) -> Texas Instruments
Connections:
- net AUX_5V: now also U2_NULL.7 (V+); no longer U2_NULL.3 (V+)
- net CH2_A_INN: no longer names the net of JP2A_INN.1 (Pin_1), R2_A3A.2, SW2_A1.2 (B)
- net CH2_A_INP: no longer names the net of JP2A_INP.1 (Pin_1), R2_A3B.2, SW2_A2.2 (B)
- net CH2_A_NIP: no longer names the net of R2_A3B.1, R2_A4.2, SW2_A2.1 (A)
- net CH2_A_OUT: no longer names the net of JP2A_OUT.1 (Pin_1), R2_A2.2, TP2_EA0.1
- net CH2_A_SUM: no longer names the net of R2_A1.2, R2_A2.1, R2_A3A.1, SW2_A1.1 (A)
- net CH2_B_GJ: no longer names the net of JP2_BG.1 (Pin_1), R2_BG.2
- net CH2_B_INN: no longer names the net of JP2B_INN.1 (Pin_1), R2_BF.2, R2_BG.1
- net CH2_B_INP: no longer names the net of JP2B_INP.1 (Pin_1), R2_BBIAS.1, R2_BIN.2
- net CH2_B_OUT: no longer names the net of JP2B_OUT.1 (Pin_1), R2_BF.1, TP2_EB0.1
- net CH2_B_SIG: no longer names the net of C2_BAC.2, R2_BDIR.2, R2_BIN.1
- net CH2_B_SIGIN: no longer names the net of C2_BAC.1, J2_BSIG.1 (In), R2_BDIR.1
- net CH2_B_V1: no longer names the net of J2_BV1.1 (Pin_1), JP2_BG.2 (Pin_2), R2_BV1.2
- net CH2_C_INN: no longer names the net of JP2C_INN.1 (Pin_1), R2_C1A.2, R2_C2.1
- net CH2_C_INP: no longer names the net of JP2C_INP.1 (Pin_1), R2_C1B.2
- net CH2_C_LOOP: no longer names the net of JP2_C.2 (Pin_2), R2_C2.2
- net CH2_C_NULLOUT: no longer names the net of C2_CNULL.1, JP2_C.1 (Pin_1), TP2_EC0.1
- net CH2_C_NULLOUT: now also U2_NULL.6; no longer U2_NULL.5
- net CH2_C_OUT: no longer names the net of JP2C_OUT.1 (Pin_1), R2_CL.1, TP2_V2.1
- net CH2_C_OUT: now also U2_NULL.3 (+); no longer U2_NULL.1 (+)
- net CH2_C_VCN: no longer names the net of C2_CNULL.2, R2_CVC.2, U2_NULL.2 (-)
- net CH2_DSIG: no longer names the net of J2_DSIG.1 (In), R2_D2.2
- net CH2_D_INJ: no longer names the net of C2_D2.2, R2_D2.1
- net CH2_D_INN: no longer names the net of C2_D1A.1, JP2D_INN.1 (Pin_1), R2_D1A.2
- net CH2_D_INP: no longer names the net of C2_D1B.1, JP2D_INP.1 (Pin_1), R2_D1B.2
- net CH2_D_OUT: no longer names the net of C2_D2.1, JP2D_OUT.1 (Pin_1), R2_D1A.1, TP2_V0.1
- net CH2_V1TERM: no longer names the net of J2_V1C.1 (Pin_1), R2_CL.2
- net CH2_VCTERM: no longer names the net of J2_VC.1 (Pin_1), R2_CVC.1
- net CH2_VQI: no longer names the net of R2_A1.1, R2_A4.1, R2_AVQI.2, TP2_VQI.1
Other:
- note added: "A / Offset and input currents"
- note added: "B / Dynamic tests and quiescent current"
- note added: "BG open: follower; closed: gain about 101. AC option: remove BDIR, fit BAC and BBIAS."
- note added: "C / Null-loop gain and output swing"
- note added: "CNULL = 22 pF is a bring-up starting point. Servo feedback passes through the chip. Do not add a local feedback resistor around the null amplifier."
- note added: "Fixture D values remain open; all D parts stay unpopulated. Generator shields return to AGND. Offset applied stimuli relative to REF."
- note added: "Guard the high-impedance A nodes with REF. Switches remain independent."
- note added: "No board placement/routing. Fixture B PD/Iq is an engineering adaptation of Method 4005."
- note removed: "A / Vos, Ib, Ios"
- note removed: "All symbols retained with DNP flags. Values await AD / ZO / frequency. Coax shield returns to AGND; stimulus referenced/offset to REF."
- note removed: "B / Slew rate, phase margin, GBW, PD/Iq"
- note removed: "BUILD: silkscreen fixture letters beside isolation jumpers. TBD and TBD-AD are intentional. No PCB placement/routing. Fixture B PD/Iq is an EDU1 engineering adaptation, not literal Figure 4005-1 conformity."
- note removed: "C / Open-loop gain and output swing"
- note removed: "Guard CH2_A_SUM, CH2_A_INN, CH2_A_NIP, CH2_A_INP with REF. No vias inside guard; no solder-mask opening. Switches independent."
- note removed: "JP2_BG open: follower; closed: gain ~101. DC coupling default. AC option: remove R2_BDIR; fit C2_BAC and R2_BBIAS."
- note removed: "JP2_C closed for retained tests. Servo feedback passes through chip. R2_CVC fitted at 0 ohm; C2_CNULL DNP. Do not add local feedback."
- moved on the sheet: C2_BAC, C2_D1A, C2_D1B, C2_D2, J2_BSIG, J2_BV1, J2_DSIG, J2_V1C, J2_VC, JP2A_INN, JP2A_INP, JP2A_OUT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
